File: hardware/OpenRX-Mono.kicad_pcb (KiCad board)
At the start: 6 copper layers, 10 x 17.3 mm, 62 parts, among them J1 Conn_Coaxial_Small, T1 0900PC16J0042001E, U1 ESP32-C3, U2 TLV75533PDQNR, U3 LR1121IMLTRT, U4 RFX2401C, U5 SKY13373-460LF, X1 CJ17-400001010B20

Commit message: Apply DroneAid rebrand and configure upstream sync
Other:
- board text added: "DroneAid"
- board text removed: "OPEN"
